Commit message: Navtest2

File: src/rm_description/urdf/sentry.urdf.xacro (robot description, xacro)
@@ -5,5 +5,4 @@
   <link name="livox_frame" />
   <link name="base_link" />
-  <link name="yaw_link" />
   <!-- 激光雷达与底盘的固定关节 -->
   <joint name="base_joint" type="fixed">
@@ -14,6 +13,14 @@
   </joint>
   <!-- 云台部分 -->
+  <link name="gimbal_odom" />
+  <joint name="gimbal_joint" type="fixed">
+    <origin xyz="0 0 0.1" rpy="0 0 0" />
+    <parent link="base_link" />
+    <child link="gimbal_odom" />
+    <axis xyz="0 0 0" />
+  </joint>
+  <link name="yaw_link" />
   <joint name="yaw_joint" type="continuous">
-    <parent link="base_link" />
+    <parent link="gimbal_odom" />
     <child link="yaw_link" />
     <axis xyz="0 0 1" />
